File: examples/niveau_piscine_pression/niveau.brd (EAGLE design)
At the start: 97.5 x 55.9 mm, 11 parts, among them IC1 MCP6241-E_P, IC2 L7805ACV, IC3 MCP3201-CI_P, J1 DCJ0202, U1 MPX2010DP, U2 D1_MINI

Commit message: Add files via upload
Parts:
- added C1: 1000µF, rcl:EB35D
- R1, R2, R3, R4: device resistor:0204V -> rcl:0309/10
Connections:
- net N$3: now also C1.-
- net N$4: now also C1.+
Routing:
- net N$2: track 10.2 -> 6.35 mm
- net N$1: track 12.8 -> 8.98 mm
- net N$5: track 76.2 -> 77.8 mm
Changed lines of the file:
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@@
 <?xml version="1.0" encoding="utf-8"?>
 <!DOCTYPE eagle SYSTEM "eagle.dtd">
-<eagle version="9.1.0">
+<eagle version="8.5.2">
 <drawing>
 <settings>
@@
 <param name="checkStop" value="0"/>
 <param name="checkValues" value="0"/>
-<param name="checkNames" value="1"/>
-<param name="checkWireStubs" value="1"/>
-<param name="checkPolygonWidth" value="0"/>
 <param name="useDiameter" value="13"/>
 <param name="maxErrors" value="50"/>
@@
 <attribute name="OC_NEWARK" value="unknown" x="90.17" y="68.58" size="1.778" layer="27" rot="R180" display="off"/>
 </element>
-<element name="R1" library="resistor" library_urn="urn:adsk.eagle:library:348" package="0204V" package3d_urn="urn:adsk.eagle:package:25948/1" value="" x="21.59" y="50.8"/>
-<element name="R2" library="resistor" library_urn="urn:adsk.eagle:library:348" package="0204V" package3d_urn="urn:adsk.eagle:package:25948/1" value="" x="21.59" y="39.37"/>
-<element name="R3" library="resistor" library_urn="urn:adsk.eagle:library:348" package="0204V" package3d_urn="urn:adsk.eagle:package:25948/1" value="" x="27.94" y="39.37" rot="R270"/>
-<element name="R4" library="resistor" library_urn="urn:adsk.eagle:library:348" package="0204V" package3d_urn="urn:adsk.eagle:package:25948/1" value="" x="27.94" y="52.07" rot="R270"/>
+<element name="R1" library="rcl" library_urn="urn:adsk.eagle:library:334" package="0309/10" package3d_urn="urn:adsk.eagle:package:23567/1" value="" x="21.59" y="50.8">
+<attribute name="SPICEPREFIX" value="R" x="21.59" y="50.8" size="1.778" layer="27" display="off"/>
+</element>
+<element name="R2" library="rcl" library_urn="urn:adsk.eagle:library:334" package="0309/10" package3d_urn="urn:adsk.eagle:package:23567/1" value="" x="21.59" y="39.37">
+<attribute name="SPICEPREFIX" value="R" x="21.59" y="39.37" size="1.778" layer="27" display="off"/>
+</element>
+<element name="R3" library="rcl" library_urn="urn:adsk.eagle:library:334" package="0309/10" package3d_urn="urn:adsk.eagle:package:23567/1" value="" x="27.94" y="39.37" rot="R270">
+<attribute name="SPICEPREFIX" value="R" x="27.94" y="39.37" size="1.778" layer="27" rot="R270" display="off"/>
+</element>
+<element name="R4" library="rcl" library_urn="urn:adsk.eagle:library:334" package="0309/10" package3d_urn="urn:adsk.eagle:package:23567/1" value="" x="27.94" y="52.07" rot="R270">
+<attribute name="SPICEPREFIX" value="R" x="27.94" y="52.07" size="1.778" layer="27" rot="R270" display="off"/>
+</element>
 <element name="U1" library="MPX2010DP" package="CASE-344C-01-ISSUE-B" value="MPX2010DP" x="10.16" y="40.64" rot="R90">
 <attribute name="ARROW_PART_NUMBER" value="MPX2010DP" x="10.16" y="40.64" size="1.778" layer="27" rot="R90" display="off"/>
@@
 </element>
 <element name="JP1" library="jumper" library_urn="urn:adsk.eagle:library:252" package="JP1" package3d_urn="urn:adsk.eagle:package:15455/1" value="" x="59.69" y="63.5" rot="R270"/>
+<element name="C1" library="rcl" library_urn="urn:adsk.eagle:library:334" package="EB35D" package3d_urn="urn:adsk.eagle:package:23395/1" value="1000µF" x="31.75" y="-1.27">
+<attribute name="SPICEPREFIX" value="C" x="31.75" y="-1.27" size="1.778" layer="27" display="off"/>
+</element>
 </elements>
 <signals>
@@
 <contactref element="IC3" pad="3"/>
 <contactref element="U2" pad="10"/>
-<wire x1="27.94" y1="53.34" x2="42.07" y2="67.47" width="0.1524" layer="1"/>
+<wire x1="27.94" y1="57.15" x2="42.07" y2="67.47" width="0.1524" layer="1"/>
 <wire x1="42.07" y1="67.47" x2="42.07" y2="72.39" width="0.1524" layer="1"/>
 <wire x1="60.96" y1="50.8" x2="88.9" y2="50.8" width="0.1524" layer="1"/>
@@
 <wire x1="24.13" y1="34.29" x2="25.4" y2="35.56" width="0.1524" layer="1" curve="90"/>
 <wire x1="25.4" y1="35.56" x2="25.4" y2="53.34" width="0.1524" layer="1"/>
-<wire x1="25.4" y1="53.34" x2="27.94" y2="53.34" width="0.1524" layer="1"/>
+<wire x1="25.4" y1="53.34" x2="27.94" y2="57.15" width="0.1524" layer="1"/>
 <wire x1="39.275" y1="45.72" x2="39.37" y2="45.72" width="0.1524" layer="1"/>
 <wire x1="39.37" y1="45.72" x2="43.18" y2="45.72" width="0.1524" layer="1"/>
@@
 <wire x1="38.1" y1="45.72" x2="36.83" y2="45.72" width="0.1524" layer="1"/>
 <wire x1="36.83" y1="45.72" x2="36.83" y2="53.34" width="0.1524" layer="1"/>
-<wire x1="36.83" y1="53.34" x2="27.94" y2="53.34" width="0.1524" layer="1"/>
+<wire x1="36.83" y1="53.34" x2="27.94" y2="57.15" width="0.1524" layer="1"/>
+<contactref element="C1" pad="-"/>
+<wire x1="36.83" y1="-1.27" x2="24.13" y2="34.29" width="0" layer="19" extent="1-1"/>
 </signal>
 <signal name="N$2">
 <contactref element="U1" pad="2"/>
 <contactref element="R2" pad="1"/>
-<wire x1="10.16" y1="39.37" x2="20.32" y2="39.37" width="0.1524" layer="1"/>
+<wire x1="10.16" y1="39.37" x2="16.51" y2="39.37" width="0.1524" layer="1"/>
 </signal>
 <signal name="N$1">
@@
 <contactref element="R1" pad="1"/>
 <wire x1="10.16" y1="44.45" x2="16.51" y2="50.8" width="0.1524" layer="1"/>
-<wire x1="16.51" y1="50.8" x2="20.32" y2="50.8" width="0.1524" layer="1"/>
 </signal>
 <signal name="N$4">
@@
 <wire x1="85.37" y1="68.58" x2="88.37" y2="71.58" width="0.1524" layer="1" curve="-90"/>
 <wire x1="88.37" y1="71.58" x2="90.17" y2="71.58" width="0.1524" layer="1"/>
+<contactref element="C1" pad="+"/>
+<wire x1="26.67" y1="-1.27" x2="10.16" y2="41.91" width="0" layer="19" extent="1-1"/>
 </signal>
 <signal name="N$6">
@@
 <wire x1="78.74" y1="34.29" x2="45.72" y2="34.29" width="0.1524" layer="1"/>
 <wire x1="31.75" y1="34.29" x2="31.75" y2="38.1" width="0.1524" layer="1"/>
-<wire x1="31.75" y1="38.1" x2="27.94" y2="38.1" width="0.1524" layer="1"/>
+<wire x1="31.75" y1="38.1" x2="27.94" y2="34.29" width="0.1524" layer="1"/>
 <wire x1="45.72" y1="34.29" x2="31.75" y2="34.29" width="0.1524" layer="1"/>
 </signal>
@@
 <contactref element="R1" pad="2"/>
 <contactref element="R3" pad="1"/>
-<wire x1="27.94" y1="40.64" x2="39.275" y2="40.64" width="0.1524" layer="1"/>
-<wire x1="22.86" y1="50.8" x2="22.86" y2="55.88" width="0.1524" layer="16"/>
+<wire x1="27.94" y1="44.45" x2="39.275" y2="40.64" width="0.1524" layer="1"/>
+<wire x1="26.67" y1="50.8" x2="22.86" y2="55.88" width="0.1524" layer="16"/>
 <wire x1="22.86" y1="55.88" x2="24.13" y2="57.15" width="0.1524" layer="16"/>
 <wire x1="24.13" y1="57.15" x2="35.56" y2="57.15" width="0.1524" layer="16"/>
 <wire x1="35.56" y1="57.15" x2="35.56" y2="48.26" width="0.1524" layer="16"/>
-<wire x1="35.56" y1="48.26" x2="27.94" y2="40.64" width="0.1524" layer="16"/>
+<wire x1="35.56" y1="48.26" x2="27.94" y2="44.45" width="0.1524" layer="16"/>
 </signal>
 <signal name="N$9">
@@
 <wire x1="39.275" y1="44.45" x2="34.29" y2="44.45" width="0.1524" layer="1"/>
 <wire x1="34.29" y1="44.45" x2="34.29" y2="50.8" width="0.1524" layer="1"/>
-<wire x1="34.29" y1="50.8" x2="27.94" y2="50.8" width="0.1524" layer="1"/>
-<wire x1="22.86" y1="39.37" x2="22.86" y2="45.72" width="0.1524" layer="16"/>
-<wire x1="22.86" y1="45.72" x2="27.94" y2="50.8" width="0.1524" layer="16"/>
+<wire x1="34.29" y1="50.8" x2="27.94" y2="46.99" width="0.1524" layer="1"/>
+<wire x1="26.67" y1="39.37" x2="22.86" y2="45.72" width="0.1524" layer="16"/>
+<wire x1="22.86" y1="45.72" x2="27.94" y2="46.99" width="0.1524" layer="16"/>
 </signal>
 <signal name="N$8">
@@
 </signal>
 </signals>
-<mfgpreviewcolors>
-<mfgpreviewcolor name="soldermaskcolor" color="0xC8008000"/>
-<mfgpreviewcolor name="silkscreencolor" color="0xFFFEFEFE"/>
-<mfgpreviewcolor name="backgroundcolor" color="0xFF282828"/>
-<mfgpreviewcolor name="coppercolor" color="0xFFFFBF00"/>
-<mfgpreviewcolor name="substratecolor" color="0xFF786E46"/>
-</mfgpreviewcolors>
 </board>
 </drawing>
